File: PCB/Left/3leaf_fall.kicad_sch (KiCad schematic)
At the start: 24 parts

Commit message: Add TC-2030 interface; generate gerbers
Parts:
- added J1: TC2030, Connector:Tag-Connect_TC2030-IDC-NL_2x03_P1.27mm_Vertical, symbol Connector:TC2030
- added SW1: SW_Reed, keeblib:Magnet_reed_switch, symbol Switch:SW_Reed
Connections:
- net GND: now also J1.5
- net SWC: now also J1.4
- net SWD: now also J1.2
- net VCC: now also J1.1, SW1.1; no longer BT1.P
- net RESET: now reaches U1.35 (P0.21/RESET)
- net RESET: now also J1.3
- new net: BT1.P, SW1.2
