File: dongle/leaf_dongle.kicad_pcb (KiCad board)
At the start: 2 copper layers, 21 x 60.4 mm, 7 parts, among them J1 UP20-C-F-G-FL-P12-TR

Commit message: Add TC-2030 interface; generate gerbers
Parts:
- added J2: TC2030, Connector:Tag-Connect_TC2030-IDC-NL_2x03_P1.27mm_Vertical, F.Cu at (122.0, 124.9)
Connections:
- U1 pad 35: unconnected-(U1-P0.21/RESET-Pad35) -> RESET
- U1 pad 36: unconnected-(U1-SWDCLK-Pad36) -> SWDCLK
- U1 pad 37: unconnected-(U1-SWDIO-Pad37) -> SWDIO
Routing:
- net -3V3: track 37.0 -> 50.9 mm, vias 2 -> 4
- net SWDCLK: track 0.00 -> 10.4 mm, vias 0 -> 2
- net SWDIO: track 0.00 -> 8.18 mm
- net RESET: track 0.00 -> 7.17 mm

Commit message: Use logic shifter on dongle
Parts:
- removed R1: 0.068, Resistor_SMD:R_0805_2012Metric
- removed R2: 0.22, Resistor_SMD:R_0805_2012Metric
- added U2: SN74LVC1T45DCK, Package_TO_SOT_SMD:SOT-363_SC-70-6, F.Cu at (129.9, 113.4)
Connections:
- D1 pad 2: NEO -> Net-(D1-DIN)
Routing:
- net NEO: track 11.6 -> 1.94 mm, vias 2 -> 0
- net Net-(D1-DIN): track 0.00 -> 8.98 mm, vias 0 -> 2
- net VCC: track 46.0 -> 50.7 mm
- net RESET: track 7.17 -> 11.5 mm, vias 0 -> 2
- net Net-(D1-VDD): track 11.8 -> 10.3 mm
- net -3V3: track 50.9 -> 49.9 mm, vias 4 -> 2

Commit message: Update dongle to have 5.1k resistor for USB power
Parts:
- added R1: 5.1k, Resistor_SMD:R_0402_1005Metric, F.Cu at (133.6, 81.3)
Connections:
- J1 pad A5: unconnected-(J1-CC1-PadA5) -> Net-(J1-CC1)
Routing:
- net Net-(J1-CC1): track 0.00 -> 5.30 mm
- net GND: track 27.9 -> 29.5 mm
